Commit message: Full poistional tracking implemented, with some bugs

File: urdf/dcam_URDF.xacro (robot description, xacro)
@@ -9,10 +9,4 @@
 	</inertial>
 	<link name="camera">
-	<collision>
-		<origin xyz="0 0 0" rpy="0 0 0" />
-		<geometry>
-			<box size="0.1 0.3 0.3" />
-		</geometry>
-	</collision>
 	<visual>
 		<origin xyz="0 0 0" rpy="0 0 0" />

Commit message: Accurate relative coordinate tracking achieved

File: urdf/dcam_URDF.xacro (robot description, xacro)
@@ -12,5 +12,5 @@
 		<origin xyz="0 0 0" rpy="0 0 0" />
 		<geometry>
-			<box size="0.1 0.3 0.3 " />
+			<box size="0.05 0.05 0.05 " />
 		</geometry>
 	</visual>
